File: kicad/parasite.kicad_sch (KiCad schematic)
At the start: 29 parts, among them Q1 MMBT3906, Q4 Q_Photo_NPN, SW1 B3U-1000P, U1 E73-2G4M08S1C, U2 SHTC3, Y1 32.768kHz

Commit message: Diode Footprint changed
Changed LL4148 to the 1N4148 variant, soldering preference.
Parts:
- D1: value LL4148 -> 1N4148W; footprint Diode_SMD:D_MiniMELF -> Diode_SMD:D_SOD-123
- RST1, SW1: footprint SW_B3U-1000P -> snapeda:SW_B3U-1000P
Changed lines of the file:
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@@
       (effects (font (size 1.27 1.27)))
     )
-    (property "Value" "LL4148" (at 63.5 112.395 0)
-      (effects (font (size 1.27 1.27)))
-    )
-    (property "Footprint" "Diode_SMD:D_MiniMELF" (at 63.5 111.125 0)
+    (property "Value" "1N4148W" (at 63.5 112.395 0)
+      (effects (font (size 1.27 1.27)))
+    )
+    (property "Footprint" "Diode_SMD:D_SOD-123" (at 63.5 111.125 0)
       (effects (font (size 1.27 1.27)) hide)
     )
@@
       (effects (font (size 1.27 1.27)) (justify left))
     )
-    (property "Footprint" "SW_B3U-1000P" (at 160.02 171.45 0)
+    (property "Footprint" "snapeda:SW_B3U-1000P" (at 160.02 171.45 0)
       (effects (font (size 1.27 1.27)) (justify left bottom) hide)
     )
@@
       (effects (font (size 1.27 1.27)) (justify left))
     )
-    (property "Footprint" "SW_B3U-1000P" (at 137.16 171.45 0)
-      (effects (font (size 1.27 1.27)) (justify left bottom) hide)
-    )
+    (property "Footprint" "snapeda:SW_B3U-1000P" (at 137.16 171.45 0)
+      (effects (font (size 1.27 1.27)) (justify left bottom) hide)
+    )

Commit message: Replaced Footprints
Replaced all 0402 footprints with 0805, moved around the routing and parts to create space.
Parts:
- C1, C2, C3, C4: footprint Capacitor_SMD:C_0402_1005Metric -> Capacitor_SMD:C_0805_2012Metric
- R1, R10, R2, R4, R6, R7, R8: footprint Resistor_SMD:R_0402_1005Metric -> Resistor_SMD:R_0805_2012Metric
Changed lines of the file:
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@@
       (effects (font (size 1.27 1.27)))
     )
-    (property "Footprint" "Resistor_SMD:R_0402_1005Metric" (at 33.02 117.348 90)
+    (property "Footprint" "Resistor_SMD:R_0805_2012Metric" (at 33.02 117.348 90)
       (effects (font (size 1.27 1.27)) hide)
     )
@@
       (effects (font (size 1.27 1.27)) (justify left))
     )
-    (property "Footprint" "Capacitor_SMD:C_0402_1005Metric" (at 73.025 120.65 0)
+    (property "Footprint" "Capacitor_SMD:C_0805_2012Metric" (at 73.025 120.65 0)
       (effects (font (size 1.27 1.27)) hide)
     )
@@
       (effects (font (size 1.27 1.27)) (justify left))
     )
-    (property "Footprint" "Resistor_SMD:R_0402_1005Metric" (at 82.042 120.65 90)
+    (property "Footprint" "Resistor_SMD:R_0805_2012Metric" (at 82.042 120.65 90)
       (effects (font (size 1.27 1.27)) hide)
     )
@@
       (effects (font (size 1.27 1.27)) (justify left))
     )
-    (property "Footprint" "Resistor_SMD:R_0402_1005Metric" (at 31.75 163.322 90)
+    (property "Footprint" "Resistor_SMD:R_0805_2012Metric" (at 31.75 163.322 90)
       (effects (font (size 1.27 1.27)) hide)
     )
@@
       (effects (font (size 1.27 1.27)) (justify left))
     )
-    (property "Footprint" "Capacitor_SMD:C_0402_1005Metric" (at 178.435 125.73 0)
+    (property "Footprint" "Capacitor_SMD:C_0805_2012Metric" (at 178.435 125.73 0)
       (effects (font (size 1.27 1.27)) hide)
     )
@@
       (effects (font (size 1.27 1.27)))
     )
-    (property "Footprint" "Resistor_SMD:R_0402_1005Metric" (at 141.732 116.84 90)
+    (property "Footprint" "Resistor_SMD:R_0805_2012Metric" (at 141.732 116.84 90)
       (effects (font (size 1.27 1.27)) hide)
     )
@@
       (effects (font (size 1.27 1.27)))
     )
-    (property "Footprint" "Resistor_SMD:R_0402_1005Metric" (at 141.478 116.84 90)
+    (property "Footprint" "Resistor_SMD:R_0805_2012Metric" (at 141.478 116.84 90)
       (effects (font (size 1.27 1.27)) hide)
     )
@@
       (effects (font (size 1.27 1.27)))
     )
-    (property "Footprint" "Resistor_SMD:R_0402_1005Metric" (at 116.078 115.57 90)
+    (property "Footprint" "Resistor_SMD:R_0805_2012Metric" (at 116.078 115.57 90)
       (effects (font (size 1.27 1.27)) hide)
     )
@@
       (effects (font (size 1.27 1.27)))
     )
-    (property "Footprint" "Resistor_SMD:R_0402_1005Metric" (at 215.138 134.62 90)
+    (property "Footprint" "Resistor_SMD:R_0805_2012Metric" (at 215.138 134.62 90)
       (effects (font (size 1.27 1.27)) hide)
     )
@@
       (effects (font (size 1.27 1.27)) (justify left))
     )
-    (property "Footprint" "Capacitor_SMD:C_0402_1005Metric" (at 91.44 24.13 0)
+    (property "Footprint" "Capacitor_SMD:C_0805_2012Metric" (at 91.44 24.13 0)
       (effects (font (size 1.27 1.27)) hide)
     )
@@
       (effects (font (size 1.27 1.27)) (justify left))
     )
-    (property "Footprint" "Capacitor_SMD:C_0402_1005Metric" (at 101.6 24.13 0)
-      (effects (font (size 1.27 1.27)) hide)
-    )
+    (property "Footprint" "Capacitor_SMD:C_0805_2012Metric" (at 101.6 24.13 0)
+      (effects (font (size 1.27 1.27)) hide)
+    )
